File: I2C-8574.sch (EAGLE design)
At the start: 89 parts, among them J1 CONNECTOR-I2CLEFT, J11 RJ12/6, J2 CONNECTOR-I2CLEFT, J5 CONNECTOR-GROVE-4P-2.0-347013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, J6 RJ12/6, J7 RJ12/6, J8 CONNECTOR-GROVE-4P-2.0-347013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, J9 RJ12/6, U1 PCF8574DW, U2 PCF8574ADW

Commit message: 3.0
Parts:
- removed C5: 150uF, SPCoast:CAP-POL0810
- removed J10: (no value), SPCoast:CONNECTOR-DC-POWER-RA
- removed J11, J6, J7, J9: RJ12/6, SPCoast:CONNECTOR-RJ25-6P6C
- removed JP1, JP4, JP5, JP6: .100x1x6, SPCoast:CONNECTOR-M06LOCK
- removed LED0, LED1, LED10, LED11, LED12, LED13, LED14, LED15, LED2, LED3, LED4, LED5, LED6, LED7, LED8, LED9: Y-0330050P1, SPCoast:LED0603-LED
- removed POWER: 7-12vDC, SPCoast-minimal:POWER_LABEL
- removed Q0, Q1, Q10, Q11, Q12, Q13, Q14, Q15, Q2, Q3, Q4, Q5, Q6, Q7, Q8, Q9: (no value), SPCoast:MOSFET-P-044021001
- removed R0, R1, R10, R11, R12, R13, R14, R2, R3, R4, R5, R6, R7, R8, R9: 2K2, SPCoast:R0805-RES
- removed R15: 2K0, SPCoast:R0805-RES
- removed VIO1, VIO2, VIO3, VIO4: jumper, SPCoast:JUMPER-3PTH-LOCK
- added FID-U1, FID-U2, FID1, FID2, FID3: FIDUCIAL, SPCoast:FIDUCIAL
- added U$2, U$3, U$4, U$5: IO4-IOBBARE, SPCoast:IO4-IOBBARE
- A1, A2, A3: device SPCoast:JUMPER-3PTH-LOCK -> SPCoast-minimal:JUMPER-3PTH-LOCK
- BOARD1: value BOARD80X100-NOHOLES -> (none)
- C1, C2, C3, C4: device SPCoast:CAP0805 -> SPCoast-minimal:C0805
- R16, R17, R18: device SPCoast:R0805-RES -> SPCoast-minimal:R0805-RES
- SCL, SDA: device SPCoast:JUMPER-2PTH_LOCK -> SPCoast-minimal:JUMPER-2PTH_LOCK
- U1: device SPCoast:PCF8574DW -> SPCoast-minimal:PCF8574DW
- U2: device SPCoast:PCF8574ADW -> SPCoast-minimal:PCF8574ADW
Connections:
- removed net N$10: LED7.A, R7.1
- removed net N$11: Q0.D, R0.2
- removed net N$12: Q5.D, R5.2
- removed net N$13: Q6.D, R6.2
- removed net N$14: Q7.D, R7.2
- removed net N$15: LED8.A, R8.1
- removed net N$16: LED9.A, R9.1
- removed net N$17: LED10.A, R10.1
- removed net N$18: Q8.D, R8.2
- removed net N$2: LED0.A, R0.1
- removed net N$22: Q9.D, R9.2
- removed net N$23: Q10.D, R10.2
- removed net N$24: Q11.D, R11.2
- removed net N$25: LED11.A, R11.1
- removed net N$26: LED14.A, R14.1
- removed net N$27: LED12.A, R12.1
- removed net N$28: LED13.A, R13.1
- removed net N$29: LED15.A, R15.1
- removed net N$3: LED1.A, R1.1
- removed net N$30: Q1.D, R1.2
- removed net N$31: Q2.D, R2.2
- removed net N$32: Q3.D, R3.2
- removed net N$33: Q12.D, R12.2
- removed net N$34: Q13.D, R13.2
- removed net N$35: Q14.D, R14.2
- removed net N$36: Q15.D, R15.2
- removed net N$4: LED2.A, R2.1
- removed net N$5: LED3.A, R3.1
- removed net N$6: LED4.A, R4.1
- removed net N$7: LED5.A, R5.1
- removed net N$8: Q4.D, R4.2
- removed net N$9: LED6.A, R6.1
- removed net VCC-IO1: J7.1, JP1.6, VIO1.2
- removed net VCC-IO2: J6.1, JP4.6, VIO2.2
- removed net VCC-IO3: J9.1, JP5.6, VIO3.2
- removed net VCC-IO4: J11.1, JP6.6, VIO4.2
- net !INT1: now also U1IC$1./INT; no longer U1U./INT
- net !INT2: now also U2IC$1./INT; no longer U2U./INT
- net +9V: now also U$2.VIN, U$3.VIN, U$4.VIN, U$5.VIN; no longer C5.+, J10.1, VIO1.3, VIO2.3, VIO3.3, VIO4.3
- net A0: now also U1IC$1.A0, U2IC$1.A0; no longer U1U.A0, U2U.A0
- net A1: now also U1IC$1.A1, U2IC$1.A1; no longer U1U.A1, U2U.A1
- net A2: now also U1IC$1.A2, U2IC$1.A2; no longer U1U.A2, U2U.A2
- net GND: now also U$2.GND, U$3.GND, U$4.GND, U$5.GND; no longer C5.-, J10.2, J10.3, J11.6, J6.6, J7.6, J9.6, JP1.1, JP4.1, JP5.1, JP6.1, LED0.C, LED1.C, LED10.C, LED11.C, LED12.C, LED13.C, LED14.C, LED15.C, LED2.C, LED3.C, LED4.C, LED5.C, LED6.C, LED7.C, LED8.C, LED9.C
- net P1: now also U$2.P1, U1IC$1.P0; no longer J7.2, JP1.5, Q0.G, U1U.P0
- net P10: now also U$4.P2, U2IC$1.P1; no longer J9.3, JP5.4, Q9.G, U2U.P1
- net P11: now also U$4.P3, U2IC$1.P2; no longer J9.4, JP5.3, Q10.G, U2U.P2
- net P12: now also U$4.P4, U2IC$1.P3; no longer J9.5, JP5.2, Q11.G, U2U.P3
- net P13: now also U$5.P1, U2IC$1.P4; no longer J11.2, JP6.5, Q12.G, U2U.P4
- net P14: now also U$5.P2, U2IC$1.P5; no longer J11.3, JP6.4, Q13.G, U2U.P5
- net P15: now also U$5.P3, U2IC$1.P6; no longer J11.4, JP6.3, Q14.G, U2U.P6
- net P16: now also U$5.P4, U2IC$1.P7; no longer J11.5, JP6.2, Q15.G, U2U.P7
- net P2: now also U$2.P2, U1IC$1.P1; no longer J7.3, JP1.4, Q1.G, U1U.P1
- net P3: now also U$2.P3, U1IC$1.P2; no longer J7.4, JP1.3, Q2.G, U1U.P2
- net P4: now also U$2.P4, U1IC$1.P3; no longer J7.5, JP1.2, Q3.G, U1U.P3
- net P5: now also U$3.P1, U1IC$1.P4; no longer J6.2, JP4.5, Q4.G, U1U.P4
- net P6: now also U$3.P2, U1IC$1.P5; no longer J6.3, JP4.4, Q5.G, U1U.P5
- net P7: now also U$3.P3, U1IC$1.P6; no longer J6.4, JP4.3, Q6.G, U1U.P6
- net P8: now also U$3.P4, U1IC$1.P7; no longer J6.5, JP4.2, Q7.G, U1U.P7
- net P9: now also U$4.P1, U2IC$1.P0; no longer J9.2, JP5.5, Q8.G, U2U.P0
- net SCL: now also U1IC$1.SCL, U2IC$1.SCL; no longer U1U.SCL, U2U.SCL
- net SDA: now also U1IC$1.SDA, U2IC$1.SDA; no longer U1U.SDA, U2U.SDA
- net VCC: now also U$2.5V, U$3.5V, U$4.5V, U$5.5V; no longer Q0.S, Q1.S, Q10.S, Q11.S, Q12.S, Q13.S, Q14.S, Q15.S, Q2.S, Q3.S, Q4.S, Q5.S, Q6.S, Q7.S, Q8.S, Q9.S, VIO1.1, VIO2.1, VIO3.1, VIO4.1
Other:
- note added: "3.0"
- note added: "Changes DFM Changes"
- note removed: "2.4"
- note removed: "Changes Made 5v/9c jumper a per port selected item Renamed from IO16-8574 to reflect generic I2C usability"
- moved on the sheet: J5, J8
